Commit message: Integration of the lamp effector to the SRDF

File: config/poppy_ergo_jr.srdf.xacro (robot description, xacro)
@@ -4,5 +4,7 @@
     A URDF file must exist for this robot as well, where the joints and the links that are referenced are defined
 -->
-<robot name="poppy_ergo_jr">
+<robot xmlns:xacro="http://www.ros.org/wiki/xacro" name="poppy_ergo_jr">
+    <xacro:arg name="lamp" default="false"/>
+    <xacro:arg name="gripper" default="false"/>
     <!--GROUPS: Representation of a set of joints and links. This can be useful for specifying DOF to plan for, defining arms, end effectors, etc-->
     <!--LINKS: When a link is specified, the parent joint of that link (if it exists) is automatically included-->
@@ -26,4 +28,5 @@
         <chain base_link="base_link" tip_link="fixed_tip" />
     </group>
+    <xacro:if value="$(arg gripper)">
     <group name="arm_and_finger">
         <link name="base_link" />
@@ -53,7 +56,20 @@
         <joint name="m6" value="0" />
     </group_state>
+    </xacro:if>
+    <xacro:if value="$(arg lamp)">
+    <group_state name="base_posture" group="arm">
+        <joint name="m1" value="0" />
+        <joint name="m2" value="0" />
+        <joint name="m3" value="0" />
+        <joint name="m4" value="0" />
+        <joint name="m5" value="0" />
+        <joint name="m6" value="0" />
+    </group_state>
+    </xacro:if>
     <!--END EFFECTOR: Purpose: Represent information about an end effector.-->
     <end_effector name="fixed_tip" parent_link="fixed_tip" group="arm" />
+    <xacro:if value="$(arg gripper)">
     <end_effector name="moving_tip" parent_link="moving_tip" group="arm_and_finger" />
+    </xacro:if>
     <!--DISABLE COLLISIONS: By default it is assumed that any link of the robot could potentially come into collision with any other link in the robot. This tag disables collision checking between a specified pair of links. -->
     <disable_collisions link1="base_link" link2="long_U" reason="Adjacent" />

Commit message: camera and gripper kind of works

File: config/poppy_ergo_jr.srdf.xacro (robot description, xacro)
@@ -12,21 +12,64 @@
     <!--CHAINS: When a chain is specified, all the links along the chain (including endpoints) are included in the group. Additionally, all the joints that are parents to included links are also included. This means that joints along the chain and the parent joint of the base link are included in the group-->
     <!--SUBGROUPS: Groups can also be formed by referencing to already defined group names-->
+    <xacro:if value="$(arg gripper)">
+    <!-- <group name="arm"> -->
+    <!--     <link name="base_link" /> -->
+    <!--     <link name="long_U" /> -->
+    <!--     <link name="section_1" /> -->
+    <!--     <link name="section_2" /> -->
+    <!--     <link name="section_3" /> -->
+    <!--     <link name="section_4" /> -->
+    <!--     <link name="fixed_tip" /> -->
+    <!--     <joint name="m1" /> -->
+    <!--     <joint name="m2" /> -->
+    <!--     <joint name="m3" /> -->
+    <!--     <joint name="m4" /> -->
+    <!--     <joint name="m5" /> -->
+    <!--     <!-\- <joint name="m6" /> -\-> -->
+    <!--     <joint name="t7f" /> -->
+    <!--     <chain base_link="base_link" tip_link="fixed_tip" /> -->
+    <!-- </group> -->
+    <!-- <group_state name="base_posture" group="arm"> -->
+    <!--     <joint name="m1" value="0" /> -->
+    <!--     <joint name="m2" value="0" /> -->
+    <!--     <joint name="m3" value="0" /> -->
+    <!--     <joint name="m4" value="0" /> -->
+    <!--     <joint name="m5" value="0" /> -->
+    <!--     <!-\- <joint name="m6" value="0" /> -\-> -->
+    <!-- </group_state> -->
     <group name="arm">
-        <link name="base_link" />
-        <link name="long_U" />
-        <link name="section_1" />
-        <link name="section_2" />
-        <link name="section_3" />
-        <link name="section_4" />
-        <link name="fixed_tip" />
-        <joint name="m1" />
-        <joint name="m2" />
-        <joint name="m3" />
-        <joint name="m4" />
-        <joint name="m5" />
-        <joint name="t7f" />
+    <!--     <joint name="m1" /> -->
+    <!--     <joint name="m2" /> -->
+    <!--     <joint name="m3" /> -->
+    <!--     <joint name="m4" /> -->
+    <!--     <joint name="m5" /> -->
+        <!-- <joint name="m6" /> -->
+    <!--     <joint name="t7f" /> -->
+        <passive_joint name="m6" />
         <chain base_link="base_link" tip_link="fixed_tip" />
     </group>
-    <xacro:if value="$(arg gripper)">
+    <!--GROUP STATES: Purpose: Define a named state for a particular group, in terms of joint values. This is useful to define states like 'folded arms'-->
+    <group_state name="base_posture" group="arm">
+        <joint name="m1" value="0" />
+        <joint name="m2" value="0" />
+        <joint name="m3" value="0" />
+        <joint name="m4" value="0" />
+        <joint name="m5" value="0" />
+        <!-- <joint name="m6" value="0" /> -->
+    </group_state>
+    <group name="finger">
+    <!--     <joint name="m1" /> -->
+    <!--     <joint name="m2" /> -->
+    <!--     <joint name="m3" /> -->
+    <!--     <joint name="m4" /> -->
+    <!--     <joint name="m5" /> -->
+        <joint name="m6" />
+    <!--     <joint name="t7f" /> -->
+        <chain base_link="section_4" tip_link="moving_tip" />
+    </group>
+    <!--GROUP STATES: Purpose: Define a named state for a particular group, in terms of joint values. This is useful to define states like 'folded arms'-->
+    <group_state name="base_posture" group="finger">
+        <joint name="m6" value="0" />
+    </group_state>
     <group name="arm_and_finger">
         <link name="base_link" />
@@ -58,4 +101,20 @@
     </xacro:if>
     <xacro:if value="$(arg lamp)">
+    <group name="arm">
+        <link name="base_link" />
+        <link name="long_U" />
+        <link name="section_1" />
+        <link name="section_2" />
+        <link name="section_3" />
+        <link name="section_4" />
+        <link name="fixed_tip" />
+        <joint name="m1" />
+        <joint name="m2" />
+        <joint name="m3" />
+        <joint name="m4" />
+        <joint name="m5" />
+        <joint name="t7f" />
+        <chain base_link="base_link" tip_link="fixed_tip" />
+    </group>
     <group_state name="base_posture" group="arm">
         <joint name="m1" value="0" />
@@ -71,6 +130,8 @@
     <xacro:if value="$(arg gripper)">
     <end_effector name="moving_tip" parent_link="moving_tip" group="arm_and_finger" />
+    <end_effector name="moving_tip" parent_link="moving_tip" group="finger" />
     </xacro:if>
     <!--DISABLE COLLISIONS: By default it is assumed that any link of the robot could potentially come into collision with any other link in the robot. This tag disables collision checking between a specified pair of links. -->
+    <disable_collisions link1="base_link" link2="ergo_jr/camera_ergo_link" reason="Adjacent" />
     <disable_collisions link1="base_link" link2="long_U" reason="Adjacent" />
     <disable_collisions link1="long_U" link2="section_1" reason="Adjacent" />
@@ -79,3 +140,6 @@
     <disable_collisions link1="section_3" link2="section_4" reason="Adjacent" />
     <disable_collisions link1="section_4" link2="section_5" reason="Adjacent" />
+    <xacro:if value="$(arg gripper)">
+    <disable_collisions link1="section_5" link2="dummy_gripper_tip" reason="Adjacent" />
+    </xacro:if>
 </robot>
